File: Schematic/STM32_WhiteBoard_64/STM32_WhiteBoard_64.kicad_pcb (KiCad board)
At the start: 2 copper layers, 25.6 x 67.6 mm, 60 parts, among them J1 SWDIO+Serial, J2 USB_B_Micro, J3 Header2, J4 Header1, Q1 BC847BS, Q2 Si3493DDV, Q3 BC857BS, SW1 Boot0, SW2 Reset, SW3 User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

Commit message: Added ESD protection for USB.
Parts:
- removed the C15 at (189.9, 90.0)
- removed C18: 75pF, Capacitor_SMD:C_0603_1608Metric_Pad1.08x0.95mm_HandSolder
- removed F1: 1A, Fuse:Fuse_1206_3216Metric_Pad1.42x1.75mm_HandSolder
- removed the R10 at (186.4, 85.6)
- removed the U4 at (190.9, 81.2)
- added C17: 10µF 16V, Capacitor_SMD:C_0603_1608Metric_Pad1.08x0.95mm_HandSolder, B.Cu at (190.5, 94.5)
- added U2: USBLC6-2P6, Retronics_IC:USBLC6-2SC6, B.Cu at (178.3, 107.5)
- added U5: TPS560430, Package_TO_SOT_SMD:SOT-23-6, B.Cu at (188.8, 81.8)
- C1: value 10µF -> 4.7µF
- C14: value 22µF 10V -> 10µF 16V
- C15: renamed from C16; value 10µF 35V -> 10µF 50V; footprint Capacitor_SMD:C_0603_1608Metric_Pad1.08x0.95mm_HandSolder -> Capacitor_SMD:C_0805_2012Metric_Pad1.18x1.45mm_HandSolder; moved to F.Cu
- FB1: value 100Ω@100MHz 30mΩ@DC -> 100Ω@100MHz
- J2: footprint digikey-footprints:USB_Micro_B_Female_10118194-0001LF -> Retronics_Connectors:USB_Micro_B_Female_10118194-0001LF
- L2: value 10µH 1A -> 6.8µH 1A; footprint Inductor_SMD:L_Taiyo-Yuden_NR-20xx_HandSoldering -> Inductor_SMD:L_1008_2520Metric_Pad1.43x2.20mm_HandSolder
- R10: renamed from R11; value 22kΩ -> 22.1kΩ
- R9: value 49.9Ω -> 51kΩ
- SW1, SW2, SW3: footprint myDevices:PTS840ESDGMSMTRLFS -> Retronics_Switches:SKTHACE010
- moved R9 9.87 mm to (194.2, 81.8), turned to 90 degrees
- moved R10 9.38 mm to (194.2, 86.3), turned to 90 degrees
- moved FB1 9.36 mm to (191.9, 86.3), turned to 90 degrees
- moved Q2 7.32 mm to (188.8, 90.5), turned to 90 degrees
- moved R12 6.03 mm to (184.9, 93.0), turned to 0 degrees
- moved C13 5.24 mm to (186.2, 81.8), turned to 90 degrees
- moved C14 4.82 mm to (188.8, 87.7), turned to 0 degrees
- moved C15 3.24 mm to (193.7, 81.8), turned to -90 degrees
- moved C16 3.10 mm to (191.5, 81.8)
- moved L2 2.70 mm to (188.8, 85.4), turned to 0 degrees
- moved D6 2.13 mm to (189.0, 81.2)
- moved D7 2.13 mm to (191.4, 81.2)
- moved Q3 1.55 mm to (184.9, 90.5), turned to 180 degrees
- moved D4 0.97 mm to (192.1, 136.2)
- moved R3 0.80 mm to (192.1, 140.4)
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- renumbered C17 to C16, R12 to R11, R13 to R12, U2 to U3, U3 to U4
Connections:
- net /PA13 renamed /PA13_SWDIO
- net /PA14 renamed /PA14_SWCLK
- net /PA2 renamed /PA2_UART2TX
- net /PA3 renamed /PA3_UART2RX
- net /PA4 renamed /PA4_CS
- net /PA5 renamed /PA5_SPI1CLK
- net /PA6 renamed /PA6_SPI1MISO
- net /PA7 renamed /PA7_SPI1MOSI
- net /PB3 renamed /PB3_SWO
- net /PC13 renamed /PC13_LED
- net /PD2 renamed /PD2_USERBTN
- FB1 pad 1: Net-(C14-Pad2) -> Net-(Q3A-E1)
- FB1 pad 2: Net-(Q3A-E1) -> Net-(C14-Pad2)
- J2 pad 2: /A11 -> /A11_USBD-
- J2 pad 3: /A12 -> /A12_USBD+
- J3 pad 1: /A11 -> /A11_USBD-
- J3 pad 2: /A12 -> /A12_USBD+
- J4 pad 2: Net-(J4-Pin_2) -> +3.3V
- R1 pad 1: +3.3V -> Net-(JP1-A)
- R10 pad 1: Net-(U4-FB) -> Net-(U5-FB)
- R9 pad 1: Net-(C14-Pad2) -> Net-(Q3A-E1)
- R9 pad 2: Net-(C18-Pad2) -> Net-(U5-FB)
- SW1 pad 1: /BOOT0 -> +3.3V
- SW1 pad 2: +3.3V -> /BOOT0
- U3 pad 44: /A11 -> Net-(U3-PA11-PWM-UART6:TX-SPI4:MISO-USB:DM)
- U3 pad 45: /A12 -> Net-(U3-PA12-UART6:RX-UART1:RTS-SPI5:MISO-USB:DP)
Routing:
- net /A11: track 38.6 -> 0.00 mm, vias 2 -> 0
- net /A12: track 38.6 -> 0.00 mm, vias 2 -> 0
- net /A11_USBD-: track 0.00 -> 33.0 mm, vias 0 -> 1
- net /A12_USBD+: track 0.00 -> 31.7 mm, vias 0 -> 1
- net VBUS: track 15.7 -> 34.1 mm, vias 0 -> 1
- net Net-(U5-FB): track 0.00 -> 11.9 mm
- net Net-(JP1-A): track 3.73 -> 10.9 mm
- net GND: track 23.3 -> 30.2 mm, vias 79 -> 71
- net Net-(U4-FB): track 6.89 -> 0.00 mm
- net Net-(C14-Pad2): track 10.9 -> 4.30 mm
- net Net-(Q3A-E1): track 9.71 -> 16.3 mm
- net Net-(Q2-G): track 10.4 -> 4.51 mm
- net Net-(U3-PA12-UART6:RX-UART1:RTS-SPI5:MISO-USB:DP): track 0.00 -> 5.52 mm, vias 0 -> 1
- net Net-(J4-Pin_2): track 4.88 -> 0.00 mm
- net Net-(C18-Pad2): track 4.44 -> 0.00 mm
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Other:
- board size 25.6 x 67.6 mm -> 25.7 x 67.6 mm
- board text added: "AREF"
- board text added: "STM32_WhiteBoard_64 R0144D_Pb_2343 Bjørner Sandom"
- board text removed: "STM32_WhiteBoard_64 R0144C_Pb_2340 Bjørner Sandom"
- board text removed: "VREF"
