File: WhiteBoard64/Schematic/STM32_WhiteBoard_64.kicad_pcb (KiCad board)
At the start: 2 copper layers, 25.7 x 67.6 mm, 58 parts, among them J1 SWDIO+Serial, J2 USB_B_Micro, J3 Header2, J4 Header1, Q1 BC847BS, Q2 Si3493DDV, Q3 BC857BS, SW1 Boot0, SW2 Reset, SW3 User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

Commit message: File cleanup
Changed lines of the file:
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@@
     (effects (font (size 1 1) (thickness 0.15)) (justify mirror))
+  )
+  (gr_text "." (at 187.9 78.9) (layer "B.SilkS")
+    (effects (font (size 1.5 1.5) (thickness 0.3) bold) (justify mirror))
   )
   (gr_text "A12" (at 175.84 82.85 270) (layer "F.SilkS" knockout)
@@
     (effects (font (size 0.8 0.8) (thickness 0.1)))
   )
-  (gr_text "." (at 191.28 92.2) (layer "F.SilkS")
-    (effects (font (size 1.5 1.5) (thickness 0.3) bold))
-  )
   (gr_text "3V3" (at 195.74 82.86 90) (layer "F.SilkS")
