File: WhiteBoard64/Schematic/STM32_WhiteBoard_64.kicad_sch (KiCad schematic)
At the start: 57 parts, among them J1 SWDIO+Serial, J2 USB_B_Micro, J3 Header2, J4 Header1, Q1 BC847BS, Q1 Si3493DDV, Q2 BC857BS, SW1 Boot0, SW2 Reset, SW3 User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

Commit message: File cleanup
Parts:
- R5: value 22.1kΩ -> 22kΩ
- R5: value 47kΩ -> 51kΩ
- R7: value 270Ω -> 330Ω
- U5: value TPS560430 -> TPS560430YFDBVR
Changed lines of the file:
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@@
       (effects (font (size 1.27 1.27)))
     )
-    (property "Value" "270Ω" (at 276.098 50.673 90)
+    (property "Value" "330Ω" (at 276.098 50.673 90)
       (effects (font (size 1.27 1.27)))
     )
@@
   (symbol (lib_id "Retronics_IC_Power:TPS560430") (at 74.93 167.64 0) (unit 1)
     (in_bom yes) (on_board yes) (dnp no) (fields_autoplaced)
-    (property "Reference" "U5" (at 74.93 158.115 0)
-      (effects (font (size 1.27 1.27)))
-    )
-    (property "Value" "TPS560430" (at 74.93 160.655 0)
+    (property "Reference" "U5" (at 74.93 157.48 0)
+      (effects (font (size 1.27 1.27)))
+    )
+    (property "Value" "TPS560430YFDBVR" (at 74.93 160.02 0)
       (effects (font (size 1.27 1.27)))
     )
@@
       (effects (font (size 1.27 1.27)) (justify left))
     )
-    (property "Value" "22.1kΩ" (at 117.0686 185.293 0)
+    (property "Value" "22kΩ" (at 117.0686 185.293 0)
       (effects (font (size 1.27 1.27)) (justify left))
     )
@@
       (effects (font (size 1.27 1.27)))
     )
-    (property "Value" "47kΩ" (at 267.589 32.385 90)
-      (effects (font (size 1.27 1.27)))
-    )
+    (property "Value" "51kΩ" (at 267.589 32.385 90)
+      (effects (font (size 1.27 1.27)))
+    )
