File: STLINK_Adapter/Schematic/STLINK_Adapter.kicad_sch (KiCad schematic)
At the start: 11 parts, among them J1 CN11, J2 CN3, J3 CN12, J4 To Nucleo STLINK Adapter, J5 IDC8, J6 FFC8

Commit message: File cleanup
Other:
- moved on the sheet: J5, J6, R1
